File: schematic/tRexRunnerNano.brd (EAGLE design)
At the start: 42 x 30 mm, 33 parts, among them IC1 MEGA88, IC2 MAX1555, T1 BC857, T2 BC847, T3 BC847, U1 TPS73033DDCR

Commit message: Small adjustments of OLED and USB connectors
- OLED connector has been moved 1mm left
- micro USB connector has been moved 1mm right
Parts:
- moved SSD1306 1.00 mm to (5.06, 22.7)
- moved USB 1.00 mm to (39.6, 23.9)
Routing:
- net USB_PWR: track 39.0 -> 40.0 mm
- net SSD1306_SCL: track 5.01 -> 6.01 mm
- net +3V3: track 59.9 -> 60.9 mm
- net SSD1306_SDA: track 11.8 -> 12.6 mm
Changed lines of the file:
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@@
 <?xml version="1.0" encoding="utf-8"?>
 <!DOCTYPE eagle SYSTEM "eagle.dtd">
-<eagle version="8.7.1">
+<eagle version="9.0.0">
 <drawing>
 <settings>
@@
 <setting verticaltext="up"/>
 </settings>
-<grid distance="10" unitdist="mil" unit="mil" style="lines" multiple="1" display="yes" altdistance="5" altunitdist="mil" altunit="mil"/>
+<grid distance="1" unitdist="mm" unit="mm" style="lines" multiple="1" display="yes" altdistance="5" altunitdist="mil" altunit="mil"/>
 <layers>
 <layer number="1" name="Top" color="4" fill="1" visible="yes" active="yes"/>
@@
 <attribute name="VALUE" x="31.877" y="28.147" size="1.27" layer="28" rot="MR270"/>
 </element>
-<element name="USB" library="SparkFun-Connectors" library_urn="urn:adsk.eagle:library:513" package="USB-MICROB" package3d_urn="urn:adsk.eagle:package:38240/1" value="AMP FCI 10103594-0001LF" x="38.608" y="23.876" smashed="yes" rot="MR180">
-<attribute name="NAME" x="37.338" y="27.686" size="1.016" layer="26" font="vector" rot="MR0"/>
-<attribute name="PROD_ID" value="CONN-09505" x="38.608" y="23.876" size="1.778" layer="28" rot="MR180" display="off"/>
-<attribute name="SF_ID" value="PRT-08533" x="38.608" y="23.876" size="1.778" layer="28" rot="MR180" display="off"/>
-<attribute name="VALUE" x="36.703" y="28.956" size="0.6096" layer="28" font="vector" ratio="20" rot="MR180" align="top-left"/>
+<element name="USB" library="SparkFun-Connectors" library_urn="urn:adsk.eagle:library:513" package="USB-MICROB" package3d_urn="urn:adsk.eagle:package:38240/1" value="AMP FCI 10103594-0001LF" x="39.608" y="23.876" smashed="yes" rot="MR180">
+<attribute name="NAME" x="38.338" y="27.686" size="1.016" layer="26" font="vector" rot="MR0"/>
+<attribute name="PROD_ID" value="CONN-09505" x="39.608" y="23.876" size="1.778" layer="28" rot="MR180" display="off"/>
+<attribute name="SF_ID" value="PRT-08533" x="39.608" y="23.876" size="1.778" layer="28" rot="MR180" display="off"/>
+<attribute name="VALUE" x="37.703" y="28.956" size="0.6096" layer="28" font="vector" ratio="20" rot="MR180" align="top-left"/>
 </element>
 <element name="C5" library="rcl" library_urn="urn:adsk.eagle:library:334" package="SMC_A" package3d_urn="urn:adsk.eagle:package:23431/1" value="1u/16V tantalum" x="32.258" y="25.734" smashed="yes" rot="MR270">
@@
 <attribute name="VALUE" x="34.035" y="19.082" size="1.27" layer="28" rot="MR0"/>
 </element>
-<element name="SSD1306" library="pinhead" library_urn="urn:adsk.eagle:library:325" package="1X04" package3d_urn="urn:adsk.eagle:package:22407/2" value="" x="6.056" y="22.686" smashed="yes" rot="R270">
-<attribute name="NAME" x="34.29" y="27.178" size="1.016" layer="25" font="vector"/>
-<attribute name="VALUE" x="2.881" y="27.766" size="1.27" layer="27" rot="R270"/>
+<element name="SSD1306" library="pinhead" library_urn="urn:adsk.eagle:library:325" package="1X04" package3d_urn="urn:adsk.eagle:package:22407/2" value="" x="5.056" y="22.686" smashed="yes" rot="R270">
+<attribute name="NAME" x="33.29" y="27.178" size="1.016" layer="25" font="vector"/>
+<attribute name="VALUE" x="1.881" y="27.766" size="1.27" layer="27" rot="R270"/>
 </element>
 <element name="VCC" library="testpad" library_urn="urn:adsk.eagle:library:385" package="TP12R" package3d_urn="urn:adsk.eagle:package:27963/1" value="TPTP12R" x="38.608" y="12.446" smashed="yes" rot="MR0">
@@
 <wire x1="27.62" y1="20.574" x2="30.734" y2="17.46" width="0.6096" layer="1"/>
 <wire x1="24.187571875" y1="20.574" x2="27.62" y2="20.574" width="0.6096" layer="1"/>
-<wire x1="7.021740625" y1="21.416" x2="6.056" y2="21.416" width="0.6096" layer="1"/>
+<wire x1="7.021740625" y1="21.416" x2="5.056" y2="21.416" width="0.6096" layer="1"/>
 <wire x1="12.24086875" y1="27.2919125" x2="12.897653125" y2="27.2919125" width="0.4064" layer="16"/>
 <wire x1="17.469659375" y1="27.2919125" x2="12.897653125" y2="27.2919125" width="0.6096" layer="1"/>
@@
 <wire x1="34.29" y1="23.114" x2="34.29" y2="25.146" width="0.4064" layer="16"/>
 <wire x1="34.29" y1="25.146" x2="33.528" y2="25.908" width="0.4064" layer="16"/>
-<wire x1="35.958" y1="25.176" x2="34.32" y2="25.176" width="0.3048" layer="16"/>
+<wire x1="36.958" y1="25.176" x2="34.32" y2="25.176" width="0.3048" layer="16"/>
 <wire x1="34.32" y1="25.176" x2="34.29" y2="25.146" width="0.1524" layer="16"/>
 <wire x1="33.528" y1="25.908" x2="33.528" y2="26.67" width="0.4064" layer="16"/>
@@
 <contactref element="IC1" pad="27"/>
 <contactref element="SSD1306" pad="1"/>
-<wire x1="6.056" y1="26.496" x2="4.286" y2="26.496" width="0.2032" layer="16"/>
-<wire x1="4.286" y1="26.496" x2="3.778" y2="25.988" width="0.2032" layer="16"/>
-<wire x1="4.46" y1="22.686" x2="3.778" y2="23.368" width="0.2032" layer="16"/>
-<wire x1="3.778" y1="25.988" x2="3.778" y2="23.368" width="0.2032" layer="16"/>
 <wire x1="9.503753125" y1="20.988396875" x2="7.80615" y2="22.686" width="0.2032" layer="16"/>
-<wire x1="7.80615" y1="22.686" x2="4.46" y2="22.686" width="0.2032" layer="16"/>
+<wire x1="3.476" y1="22.686" x2="2.794" y2="23.368" width="0.2032" layer="16"/>
+<wire x1="2.794" y1="23.368" x2="2.794" y2="25.654" width="0.2032" layer="16"/>
+<wire x1="2.794" y1="25.654" x2="3.636" y2="26.496" width="0.2032" layer="16"/>
+<wire x1="7.80615" y1="22.686" x2="3.476" y2="22.686" width="0.2032" layer="16"/>
+<wire x1="3.636" y1="26.496" x2="5.056" y2="26.496" width="0.2032" layer="16"/>
 </signal>
 <signal name="N$4">
@@
 <contactref element="IC1" pad="28"/>
 <wire x1="10.0694375" y1="21.55408125" x2="7.66751875" y2="23.956" width="0.2032" layer="16"/>
-<wire x1="7.66751875" y1="23.956" x2="6.056" y2="23.956" width="0.2032" layer="16"/>
+<wire x1="7.66751875" y1="23.956" x2="5.056" y2="23.956" width="0.2032" layer="16"/>
 </signal>
 <signal name="DUCKING_BUTTON">

Commit message: Schematic: Changes D3 to 2V7
Parts:
- D3: value LL4148 -> 2V7
Changed lines of the file:
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@@
 <attribute name="VALUE" x="21.336" y="6.858" size="1.27" layer="28" rot="MR90"/>
 </element>
-<element name="D3" library="diode" library_urn="urn:adsk.eagle:library:210" package="SOD80C" package3d_urn="urn:adsk.eagle:package:43405/2" value="LL4148" x="14.478" y="3.81" smashed="yes" rot="MR270">
+<element name="D3" library="diode" library_urn="urn:adsk.eagle:library:210" package="SOD80C" package3d_urn="urn:adsk.eagle:package:43405/2" value="2V7" x="14.478" y="3.81" smashed="yes" rot="MR270">
 <attribute name="NAME" x="17.272" y="1.27" size="1.016" layer="26" font="vector" rot="MR0"/>
 <attribute name="VALUE" x="16.891" y="5.334" size="1.27" layer="28" rot="MR270"/>

Commit message: Board: Repositions oled connector, usb and buttons
Parts:
- moved SSD1306 1.50 mm to (3.56, 22.7)
- moved DUCKING 0.75 mm to (34.0, 5.08)
- moved USB 0.25 mm to (39.9, 23.9)
Routing:
- net SSD1306_SDA: track 12.6 -> 14.1 mm
- net SSD1306_SCL: track 6.01 -> 7.51 mm
- net +3V3: track 60.9 -> 62.4 mm
- net DUCKING_BUTTON: track 18.1 -> 18.9 mm
Changed lines of the file:
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@@
 <?xml version="1.0" encoding="utf-8"?>
 <!DOCTYPE eagle SYSTEM "eagle.dtd">
-<eagle version="9.0.0">
+<eagle version="8.7.1">
 <drawing>
 <settings>
@@
 <setting verticaltext="up"/>
 </settings>
-<grid distance="1" unitdist="mm" unit="mm" style="lines" multiple="1" display="yes" altdistance="5" altunitdist="mil" altunit="mil"/>
+<grid distance="0.5" unitdist="mm" unit="mm" style="lines" multiple="1" display="yes" altdistance="5" altunitdist="mil" altunit="mil"/>
 <layers>
 <layer number="1" name="Top" color="4" fill="1" visible="yes" active="yes"/>
@@
 <attribute name="VALUE" x="31.877" y="28.147" size="1.27" layer="28" rot="MR270"/>
 </element>
-<element name="USB" library="SparkFun-Connectors" library_urn="urn:adsk.eagle:library:513" package="USB-MICROB" package3d_urn="urn:adsk.eagle:package:38240/1" value="AMP FCI 10103594-0001LF" x="39.608" y="23.876" smashed="yes" rot="MR180">
-<attribute name="NAME" x="38.338" y="27.686" size="1.016" layer="26" font="vector" rot="MR0"/>
-<attribute name="PROD_ID" value="CONN-09505" x="39.608" y="23.876" size="1.778" layer="28" rot="MR180" display="off"/>
-<attribute name="SF_ID" value="PRT-08533" x="39.608" y="23.876" size="1.778" layer="28" rot="MR180" display="off"/>
-<attribute name="VALUE" x="37.703" y="28.956" size="0.6096" layer="28" font="vector" ratio="20" rot="MR180" align="top-left"/>
+<element name="USB" library="SparkFun-Connectors" library_urn="urn:adsk.eagle:library:513" package="USB-MICROB" package3d_urn="urn:adsk.eagle:package:38240/1" value="AMP FCI 10103594-0001LF" x="39.862" y="23.876" smashed="yes" rot="MR180">
+<attribute name="NAME" x="38.592" y="27.686" size="1.016" layer="26" font="vector" rot="MR0"/>
+<attribute name="PROD_ID" value="CONN-09505" x="39.862" y="23.876" size="1.778" layer="28" rot="MR180" display="off"/>
+<attribute name="SF_ID" value="PRT-08533" x="39.862" y="23.876" size="1.778" layer="28" rot="MR180" display="off"/>
+<attribute name="VALUE" x="37.957" y="28.956" size="0.6096" layer="28" font="vector" ratio="20" rot="MR180" align="top-left"/>
 </element>
 <element name="C5" library="rcl" library_urn="urn:adsk.eagle:library:334" package="SMC_A" package3d_urn="urn:adsk.eagle:package:23431/1" value="1u/16V tantalum" x="32.258" y="25.734" smashed="yes" rot="MR270">
@@
 <attribute name="VALUE" x="10.922" y="10.16" size="1.27" layer="27" ratio="10" rot="R180"/>
 </element>
-<element name="DUCKING" library="switch-omron" library_urn="urn:adsk.eagle:library:377" package="B3F-10XX" package3d_urn="urn:adsk.eagle:package:27496/1" value="" x="33.274" y="5.08" smashed="yes">
-<attribute name="MF" value="" x="33.274" y="5.08" size="1.778" layer="27" display="off"/>
-<attribute name="MPN" value="B3F-1000" x="33.274" y="5.08" size="1.778" layer="27" display="off"/>
-<attribute name="NAME" x="29.972" y="8.556" size="1.016" layer="25" font="vector"/>
-<attribute name="OC_FARNELL" value="176432" x="33.274" y="5.08" size="1.778" layer="27" display="off"/>
-<attribute name="OC_NEWARK" value="36M3542" x="33.274" y="5.08" size="1.778" layer="27" display="off"/>
-<attribute name="VALUE" x="30.226" y="0" size="1.27" layer="27" ratio="10"/>
+<element name="DUCKING" library="switch-omron" library_urn="urn:adsk.eagle:library:377" package="B3F-10XX" package3d_urn="urn:adsk.eagle:package:27496/1" value="" x="34.02" y="5.08" smashed="yes">
+<attribute name="MF" value="" x="34.02" y="5.08" size="1.778" layer="27" display="off"/>
+<attribute name="MPN" value="B3F-1000" x="34.02" y="5.08" size="1.778" layer="27" display="off"/>
+<attribute name="NAME" x="30.718" y="8.556" size="1.016" layer="25" font="vector"/>
+<attribute name="OC_FARNELL" value="176432" x="34.02" y="5.08" size="1.778" layer="27" display="off"/>
+<attribute name="OC_NEWARK" value="36M3542" x="34.02" y="5.08" size="1.778" layer="27" display="off"/>
+<attribute name="VALUE" x="30.972" y="0" size="1.27" layer="27" ratio="10"/>
 </element>
 <element name="D1" library="diode" library_urn="urn:adsk.eagle:library:210" package="SOD323_ST" package3d_urn="urn:adsk.eagle:package:43461/1" value="BAT43WS" x="32.385" y="19.304" smashed="yes" rot="MR0">
@@
 <attribute name="VALUE" x="34.035" y="19.082" size="1.27" layer="28" rot="MR0"/>
 </element>
-<element name="SSD1306" library="pinhead" library_urn="urn:adsk.eagle:library:325" package="1X04" package3d_urn="urn:adsk.eagle:package:22407/2" value="" x="5.056" y="22.686" smashed="yes" rot="R270">
-<attribute name="NAME" x="33.29" y="27.178" size="1.016" layer="25" font="vector"/>
-<attribute name="VALUE" x="1.881" y="27.766" size="1.27" layer="27" rot="R270"/>
+<element name="SSD1306" library="pinhead" library_urn="urn:adsk.eagle:library:325" package="1X04" package3d_urn="urn:adsk.eagle:package:22407/2" value="" x="3.556" y="22.686" smashed="yes" rot="R270">
+<attribute name="NAME" x="31.79" y="27.178" size="1.016" layer="25" font="vector"/>
+<attribute name="VALUE" x="0.381" y="27.766" size="1.27" layer="27" rot="R270"/>
 </element>
 <element name="VCC" library="testpad" library_urn="urn:adsk.eagle:library:385" package="TP12R" package3d_urn="urn:adsk.eagle:package:27963/1" value="TPTP12R" x="38.608" y="12.446" smashed="yes" rot="MR0">
@@
 <wire x1="27.62" y1="20.574" x2="30.734" y2="17.46" width="0.6096" layer="1"/>
 <wire x1="24.187571875" y1="20.574" x2="27.62" y2="20.574" width="0.6096" layer="1"/>
-<wire x1="7.021740625" y1="21.416" x2="5.056" y2="21.416" width="0.6096" layer="1"/>
+<wire x1="7.021740625" y1="21.416" x2="3.556" y2="21.416" width="0.6096" layer="1"/>
 <wire x1="12.24086875" y1="27.2919125" x2="12.897653125" y2="27.2919125" width="0.4064" layer="16"/>
 <wire x1="17.469659375" y1="27.2919125" x2="12.897653125" y2="27.2919125" width="0.6096" layer="1"/>
@@
 <wire x1="34.29" y1="23.114" x2="34.29" y2="25.146" width="0.4064" layer="16"/>
 <wire x1="34.29" y1="25.146" x2="33.528" y2="25.908" width="0.4064" layer="16"/>
-<wire x1="36.958" y1="25.176" x2="34.32" y2="25.176" width="0.3048" layer="16"/>
+<wire x1="37.212" y1="25.176" x2="34.32" y2="25.176" width="0.3048" layer="16"/>
 <wire x1="34.32" y1="25.176" x2="34.29" y2="25.146" width="0.1524" layer="16"/>
 <wire x1="33.528" y1="25.908" x2="33.528" y2="26.67" width="0.4064" layer="16"/>
@@
 <contactref element="SSD1306" pad="1"/>
 <wire x1="9.503753125" y1="20.988396875" x2="7.80615" y2="22.686" width="0.2032" layer="16"/>
-<wire x1="3.476" y1="22.686" x2="2.794" y2="23.368" width="0.2032" layer="16"/>
-<wire x1="2.794" y1="23.368" x2="2.794" y2="25.654" width="0.2032" layer="16"/>
-<wire x1="2.794" y1="25.654" x2="3.636" y2="26.496" width="0.2032" layer="16"/>
-<wire x1="7.80615" y1="22.686" x2="3.476" y2="22.686" width="0.2032" layer="16"/>
-<wire x1="3.636" y1="26.496" x2="5.056" y2="26.496" width="0.2032" layer="16"/>
+<wire x1="1.976" y1="22.686" x2="1.294" y2="23.368" width="0.2032" layer="16"/>
+<wire x1="1.294" y1="23.368" x2="1.294" y2="25.654" width="0.2032" layer="16"/>
+<wire x1="1.294" y1="25.654" x2="2.136" y2="26.496" width="0.2032" layer="16"/>
+<wire x1="7.80615" y1="22.686" x2="1.976" y2="22.686" width="0.2032" layer="16"/>
+<wire x1="2.136" y1="26.496" x2="3.556" y2="26.496" width="0.2032" layer="16"/>
 </signal>
 <signal name="N$4">
@@
 <contactref element="IC1" pad="28"/>
 <wire x1="10.0694375" y1="21.55408125" x2="7.66751875" y2="23.956" width="0.2032" layer="16"/>
-<wire x1="7.66751875" y1="23.956" x2="5.056" y2="23.956" width="0.2032" layer="16"/>
+<wire x1="7.66751875" y1="23.956" x2="3.556" y2="23.956" width="0.2032" layer="16"/>
 </signal>
 <signal name="DUCKING_BUTTON">
@@
 <wire x1="17.78" y1="14.97489375" x2="17.78" y2="12.954" width="0.2032" layer="16"/>
 <wire x1="17.78" y1="12.954" x2="23.3934" y2="7.3406" width="0.2032" layer="1"/>
-<wire x1="23.3934" y1="7.3406" x2="30.0228" y2="7.3406" width="0.2032" layer="1"/>
+<wire x1="23.3934" y1="7.3406" x2="30.7688" y2="7.3406" width="0.2032" layer="1"/>
 </signal>
 </signals>
