File: hardware/tRexRunnerNano.kicad_sch (KiCad schematic)
At the start: 32 parts, among them IC1 TPS2112APWR, IC2 MAX1555EZK_T, IC3 TPS73033DBVR, IC4 CH32V003F4P6, J1 CHG, J2 BATT, J3 OLED, Q1 BC847, Q2 BC857, Q3 BC847, SW1 DUCK, SW2 JUMP

Commit message: Fix BC8x7 transistor pinouts and TPS2112A configuration
- Update PCB version to v1.0.1.
- Fix BC847 and BC857 footprints to match correct B-E-C layout.
- Connect TPS2112APWR VSNS pin to GND for proper mode selection.
- Add current-limiting resistor to TPS2112APWR ILIM pin.
Parts:
- removed Q1, Q3: BC847, Package_TO_SOT_SMD:SOT-23, symbol Simulation_SPICE:NPN
- removed Q2: BC857, Package_TO_SOT_SMD:SOT-23, symbol Simulation_SPICE:PNP
- added Q1, Q3: BC847, Package_TO_SOT_SMD:SOT-23, symbol Transistor_BJT:BC847
- added Q2: BC857, Package_TO_SOT_SMD:SOT-23, symbol Transistor_BJT:BC857
- added R9: 470, Resistor_SMD:R_0603_1608Metric, symbol Device:R
- R4, R5: value 10k -> 100k
Connections:
- net +BATT: now also Q2.2 (E)
- net GND: now also IC1.3 (VSNS), Q1.2 (E), Q3.2 (E), R9.2
- net JUMP_BTN: now also Q3.3 (C)
- net VDD: now also Q2.3 (C)
- net at R7.2, R8.1: now also Q2.1 (B)
- net at D1.1 (K): now also Q1.3 (C)
- net at R6.2: now also Q1.1 (B)
- net at SW2.2: now also Q3.1 (B)
- net at IC1.4 (ILIM): now also R9.1
- no-connect marks 17 -> 15
