File: hardware/tRexRunnerNano.kicad_sch (KiCad schematic)
At the start: 33 parts, among them IC1 TPS2112APWR, IC2 MAX1555EZK_T, IC3 TPS73033DBVR, IC4 CH32V003F4P6, J1 CHG, J2 BATT, J3 OLED, Q1 BC847, Q2 BC857, Q3 BC847, SW1 DUCK, SW2 JUMP

Commit message: Change value of C7 to 10uF
Based on the datasheet (5.3 Recommended Operating Conditions) output
capacitor's nominal value is 10uF.
Parts:
- C7: value 2u2 -> 10u
Changed lines of the file:
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@@
 			)
 		)
-		(property "Value" "2u2"
+		(property "Value" "10u"
 			(at 205.74 130.8099 0)
 			(show_name no)
